Commit message: changed urdf file remove camera for fixing

File: templates/simple_robot.urdf (robot description, URDF)
Before this commit: robot simple_robot, 4 links, 3 joints
Links:
- removed link head_link
- removed link left_leg_link
- removed link right_leg_link
- added link bicep_link, mass 0.29331; collision mesh filename=package://reactor_description/meshes/bicep_link_hull.STL; visual mesh filename=package://reactor_description/meshes/bicep_link.STL
- added link finger_link_1, mass 0.0078621; collision mesh filename=package://reactor_description/meshes/finger_link_hull.STL; visual mesh filename=package://reactor_description/meshes/finger_link.STL
- added link finger_link_2, mass 0.0078621; collision mesh filename=package://reactor_description/meshes/finger_link_hull.STL; visual mesh filename=package://reactor_description/meshes/finger_link.STL
- added link forearm_link, mass 0.138705662443181; collision mesh filename=package://reactor_description/meshes/forearm_link_hull.STL; visual mesh filename=package://reactor_description/meshes/forearm_link.STL
- added link shoulder_link, mass 0.069055; collision mesh filename=package://reactor_description/meshes/shoulder_link_hull.STL; visual mesh filename=package://reactor_description/meshes/shoulder_link.STL
- added link wrist_1, mass 0.0605067986491363; collision mesh filename=package://reactor_description/meshes/wrist_1_hull.STL; visual mesh filename=package://reactor_description/meshes/wrist_1.STL
- added link wrist_2, mass 0.0648521292346638; collision mesh filename=package://reactor_description/meshes/wrist_2_hull.STL; visual mesh filename=package://reactor_description/meshes/wrist_2.STL
- link base_link: mass 1.0 -> 0.33742; geometry collision mesh filename=package://reactor_description/meshes/base_link_hull.STL; visual mesh filename=package://reactor_description/meshes/base_link.STL
Joints:
- removed joint base_to_head
- removed joint base_to_left_leg
- removed joint base_to_right_leg
- added joint elbow_pitch: type revolute, parent bicep_link, child forearm_link, origin xyz=-0.1445 0 0.0385 rpy=0 0 0, axis 0 1 0, limit lower=-3.141593 upper=0 effort=3.0 velocity=6.178465545
- added joint finger_joint: type prismatic, parent wrist_2, child finger_link_1, origin xyz=0.088882 -0.0187500 0.0012072 rpy=1.5708 -1.5572 -3.1416, axis 0 0 1, limit lower=0 upper=0.014 effort=1.5 velocity=0.01
- added joint finger_joint_2: type prismatic, parent wrist_2, child finger_link_2, origin xyz=0.088882 0.0187500 0.0012072 rpy=1.5708 1.5572 -1.4508E-15, axis 0 0 1, limit lower=0 upper=0.014 effort=1.5 velocity=0.01, mimic joint=finger_joint
- added joint shoulder_pitch: type revolute, parent shoulder_link, child bicep_link, origin xyz=0 0 0.0265 rpy=0 0 0, axis 0 1 0, limit lower=0 upper=3.141593 effort=3.0 velocity=6.178465545
- added joint shoulder_yaw: type revolute, parent base_link, child shoulder_link, origin xyz=0 0 0.081 rpy=0 0 0, axis 0 0 1, limit lower=-3.141593 upper=3.141593 effort=1.5 velocity=6.178465545
- added joint wrist_pitch: type revolute, parent forearm_link, child wrist_1, origin xyz=0.1535 0 0 rpy=0 0 0, axis 0 1 0, limit lower=-1.57079632679 upper=1.57079632679 effort=1.5 velocity=6.178465545
- added joint wrist_roll: type revolute, parent wrist_1, child wrist_2, origin xyz=0.071 0.00175 0 rpy=0 0 0, axis 1 0 0, limit lower=-3.141593 upper=3.141593 effort=1.5 velocity=6.178465545
