Commit message: last fix

File: public/robots/robotiq_arg85_description.URDF (robot description, URDF)
Before this commit: robot robotiq_arg85_description, 9 links, 8 joints
Links:
- link left_inner_finger: geometry collision mesh filename=package://robotiq_arg85_description/../meshes/inner_finger_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; visual mesh filename=package://robotiq_arg85_description/../meshes/inner_finger_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
- link left_inner_knuckle: geometry collision mesh filename=package://robotiq_arg85_description/../meshes/inner_knuckle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; visual mesh filename=package://robotiq_arg85_description/../meshes/inner_knuckle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
- link left_outer_finger: geometry collision mesh filename=package://robotiq_arg85_description/../meshes/outer_finger_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; visual mesh filename=package://robotiq_arg85_description/../meshes/outer_finger_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
- link left_outer_knuckle: geometry collision mesh filename=package://robotiq_arg85_description/../meshes/outer_knuckle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; visual mesh filename=package://robotiq_arg85_description/../meshes/outer_knuckle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
- link right_inner_finger: geometry collision mesh filename=package://robotiq_arg85_description/../meshes/inner_finger_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; visual mesh filename=package://robotiq_arg85_description/../meshes/inner_finger_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
- link right_inner_knuckle: geometry collision mesh filename=package://robotiq_arg85_description/../meshes/inner_knuckle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; visual mesh filename=package://robotiq_arg85_description/../meshes/inner_knuckle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
- link right_outer_finger: geometry collision mesh filename=package://robotiq_arg85_description/../meshes/outer_finger_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; visual mesh filename=package://robotiq_arg85_description/../meshes/outer_finger_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
- link right_outer_knuckle: geometry collision mesh filename=package://robotiq_arg85_description/../meshes/outer_knuckle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; visual mesh filename=package://robotiq_arg85_description/../meshes/outer_knuckle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
- link robotiq_85_base_link: geometry collision mesh filename=package://robotiq_arg85_description/../meshes/robotiq_85_ba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; visual mesh filename=package://robotiq_arg85_description/../meshes/robotiq_85_ba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
